Commit message: added laser

File: my_rb1_description/urdf/my_rb1_robot.urdf (robot description, URDF)
Before this commit: robot rb1_robot, 6 links, 5 joints
Links:
- added link front_laser, mass 0.1; collision box size=0.015 0.015 0.015; visual box size=0.015 0.015 0.015

Commit message: urdf laser plugin added

File: my_rb1_description/urdf/my_rb1_robot.urdf (robot description, URDF)
Before this commit: robot rb1_robot, 7 links, 5 joints
Links:
- link front_laser: mass 0.1 -> 0.5; geometry collision cylinder length=0.20 radius=0.15; visual cylinder length=0.20 radius=0.15
Joints:
- added joint front_laser_joint: type fixed, parent base_link, child front_laser, origin xyz=0.25 0.0 0.075 rpy=3.14159 0 0
- joint back_caster_wheel_joint: axis 0 1 0 -> 1 0 0
- joint front_caster_wheel_joint: axis 0 1 0 -> 1 0 0

Commit message: modified joints for forward x movement

File: my_rb1_description/urdf/my_rb1_robot.urdf (robot description, URDF)
Before this commit: robot rb1_robot, 7 links, 6 joints
Links:
- link front_laser: geometry collision cylinder length=0.07 radius=0.05; visual cylinder length=0.07 radius=0.05
Joints:
- joint left_wheel_joint: axis 0 0 1 -> 0 0 -1
- joint right_wheel_joint: axis 0 0 1 -> 0 0 -1

Commit message: updated colours to robot

File: my_rb1_description/urdf/my_rb1_robot.urdf (robot description, URDF)
Before this commit: robot rb1_robot, 7 links, 6 joints
Links:
- removed link back_caster_wheel
- removed link front_caster_wheel
- added link back_caster, mass 0.2; collision sphere radius=0.025; visual sphere radius=0.025
- added link front_caster, mass 0.2; collision sphere radius=0.025; visual sphere radius=0.025
- link base_footprint: mass 25.0 -> None; geometry 
- link base_link: geometry collision cylinder length=0.30 radius=0.25; visual cylinder length=0.30 radius=0.25
Joints:
- removed joint back_caster_wheel_joint
- removed joint front_caster_wheel_joint
- added joint back_caster_joint: type fixed, parent base_link, child back_caster, origin xyz=-0.1 0.0 -0.15 rpy=0 0 0
- added joint front_caster_joint: type fixed, parent base_link, child front_caster, origin xyz=0.1 0.0 -0.15 rpy=0 0 0

Commit message: updated robot caster wheels to revolute reduced shaking

File: my_rb1_description/urdf/my_rb1_robot.urdf (robot description, URDF)
Before this commit: robot rb1_robot, 7 links, 6 joints
Joints:
- joint back_caster_joint: axis (none) -> 0 0 1; limit (none) -> lower=-3.1416 upper=3.1416 effort=0.0 velocity=0.0; type fixed -> revolute
- joint front_caster_joint: axis (none) -> 0 0 1; limit (none) -> lower=-3.1416 upper=3.1416 effort=0.0 velocity=0.0; type fixed -> revolute
